Commit message: Robot Urdf Added

File: my_moveit/urdf/robot.urdf (robot description, URDF)
Before this commit: robot m2wr, 12 links, 11 joints
Links:
- link arm_link_01: geometry collision cylinder length=0.70 radius=0.04; visual cylinder length=0.70 radius=0.04
- link arm_link_02: geometry collision cylinder length=0.6 radius=0.04; visual cylinder length=0.6 radius=0.04
Joints:
- joint arm_joint_02: origin xyz=0 0 0.25 rpy=0 0 0 -> xyz=0 0 0.65 rpy=0 0 0
- joint arm_joint_03: origin xyz=0 0 0.50 rpy=0 0 0 -> xyz=0 0 0.60 rpy=0 0 0

Commit message: my_aruco package added

File: my_moveit/urdf/robot.urdf (robot description, URDF)
Before this commit: robot m2wr, 12 links, 11 joints
Joints:
- joint joint_left_wheel: origin xyz=-0.05 -0.15 0 rpy=0 0 0 -> xyz=-0.20 -0.15 0 rpy=0 0 0
- joint joint_right_wheel: origin xyz=-0.05 0.15 0 rpy=0 0 0 -> xyz=-0.20 0.15 0 rpy=0 0 0
